File: Projet PCB KiCad/Projet PCB kiCad/Projet PCB kiCad.kicad_pcb (KiCad board)
At the start: 2 copper layers, 29 parts, among them J1 Conn_01x02, J2 Conn_01x02, J3 Conn_01x02, J5 Conn_01x09_Pin, J6 Conn_02x05_Top_Bottom, U1 STM32L021K4Tx, U2 BU33SD5WG-TR, U3 MCP4801, U4 STM32G431K8Tx

Commit message: Kicad fin schema
Parts:
- added IC1: M95512-RMN6TP, Package_SO:SOIC-8_3.9x4.9mm_P1.27mm, F.Cu at (191.0, 91.8)
- moved C5 17.2 mm to (171.0, 70.0)
- moved H3 17.2 mm to (165.2, 76.6)
- moved U2 17.2 mm to (185.2, 79.1)
- moved C2 17.2 mm to (171.0, 62.5)
- moved J1 17.2 mm to (176.6, 62.1)
- moved C1 17.2 mm to (171.0, 60.0)
- moved C10 17.2 mm to (171.0, 82.5)
- moved C3 17.2 mm to (171.0, 65.0)
- moved C4 17.2 mm to (171.0, 67.5)
- moved C6 17.2 mm to (171.0, 72.5)
- moved C7 17.2 mm to (171.0, 75.0)
- moved C8 17.2 mm to (171.0, 77.5)
- moved C9 17.2 mm to (171.0, 80.0)
- moved D1 17.2 mm to (189.4, 77.6)
- moved D2 17.2 mm to (189.4, 79.3)
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Connections:
- J5 pad 1: unconnected-(J5-Pin_1-Pad1) -> INT
- J5 pad 2: unconnected-(J5-Pin_2-Pad2) -> I2C_RST
- J5 pad 3: unconnected-(J5-Pin_3-Pad3) -> SDA
- J5 pad 4: unconnected-(J5-Pin_4-Pad4) -> SCL
- J5 pad 5: unconnected-(J5-Pin_5-Pad5) -> LPn
- J5 pad 6: unconnected-(J5-Pin_6-Pad6) -> PWR_EN
- J5 pad 7: unconnected-(J5-Pin_7-Pad7) -> AVDD
- J5 pad 9: unconnected-(J5-Pin_9-Pad9) -> GND
