File: Projet PCB KiCad/Projet PCB kiCad/Projet PCB kiCad.kicad_sch (KiCad schematic)
At the start: 25 parts, among them J1 Conn_01x02, J2 Conn_01x02, J3 Conn_01x02, J5 Conn_01x09_Pin, J6 Conn_02x05_Top_Bottom, U2 BU33SD5WG-TR, U4 STM32G431K8Tx

Commit message: kicad eeprom
Parts:
- added IC1: M95512-RMN6TP, SOIC127P600X175-8N, symbol M95512-RMN6TP:M95512-RMN6TP
Changed lines of the file:
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@@
+	)
+	(symbol
+		(lib_id "M95512-RMN6TP:M95512-RMN6TP")
+		(at 149.86 57.15 0)
+		(unit 1)
+		(exclude_from_sim no)
+		(in_bom yes)
+		(on_board yes)
+		(dnp no)
+		(fields_autoplaced yes)
+		(property "Reference" "IC1"
+			(at 163.83 49.53 0)
+			(effects
+				(font
+					(size 1.27 1.27)
+				)
+			)
+		)
+		(property "Value" "M95512-RMN6TP"
+			(at 163.83 52.07 0)
+			(effects
+				(font
+					(size 1.27 1.27)
+				)
+			)
+		)
+		(property "Footprint" "SOIC127P600X175-8N"
+			(at 173.99 152.07 0)
+			(effects
+				(font
+					(size 1.27 1.27)
+				)
+				(justify left top)
+				(hide yes)
+			)
+		)
+		(property "Datasheet" "https://www.st.com/resource/en/datasheet/m95512-w.pdf"
+			(at 173.99 252.07 0)
+			(effects
+				(font
+					(size 1.27 1.27)
+				)
+				(justify left top)
+				(hide yes)
+			)
+		)
+		(property "Description" "512 Kbit SPI bus EEPROM with high-speed clock"
+			(at 149.86 57.15 0)
+			(effects
+				(font
+					(size 1.27 1.27)
+				)
+				(hide yes)
+			)
+		)
+		(property "Height" "1.75"
+			(at 173.99 452.07 0)
+			(effects
+				(font
+					(size 1.27 1.27)
+				)
+				(justify left top)
+				(hide yes)
+			)
+		)
+		(property "Mouser Part Number" "511-M95512-RMN6TP"
+			(at 173.99 552.07 0)
+			(effects
+				(font
+					(size 1.27 1.27)
+				)
+				(justify left top)
+				(hide yes)
+			)
+		)
+		(property "Mouser Price/Stock" "https://www.mouser.co.uk/ProductDetail/STMicroelectronics/M95512-RMN6TP?qs=D3O9yD6Cgx9SaimnKH25jA%3D%3D"
+			(at 173.99 652.07 0)
+			(effects
+				(font
+					(size 1.27 1.27)
+				)
+				(justify left top)
+				(hide yes)
+			)
+		)
+		(property "Manufacturer_Name" "STMicroelectronics"
+			(at 173.99 752.07 0)
+			(effects
+				(font
+					(size 1.27 1.27)
+				)
+				(justify left top)
+				(hide yes)
+			)
+		)
+		(property "Manufacturer_Part_Number" "M95512-RMN6TP"
+			(at 173.99 852.07 0)
+			(effects
+				(font
+					(size 1.27 1.27)
+				)
+				(justify left top)
+				(hide yes)
+			)
+		)
+		(pin "2"
+		)
+		(pin "3"
+		)
+		(pin "4"
+		)
+		(pin "8"
+		)
+		(pin "7"
+		)
+		(pin "5"
+		)
+		(pin "6"
+		)
+		(pin "1"
+		)
+		(instances
+			(project "Projet PCB kiCad"
+				(path "/f1a28d28-fa55-4b6b-89d5-871b1ed8503e"
+					(reference "IC1")
+					(unit 1)
+				)
+			)
+		)
 	)
 	(symbol

Commit message: ajout des datasheet
Parts:
- IC1: footprint SOIC127P600X175-8N -> Package_SO:SOIC-8_3.9x4.9mm_P1.27mm
Other:
- note added: "EEPROM M95512-RMN6TP"
- note removed: "DAC MDP4801"
Changed lines of the file:
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@@
 		)
 	)
-	(text "DAC MDP4801\n"
+	(text "EEPROM M95512-RMN6TP\n"
 		(exclude_from_sim no)
-		(at 148.336 36.576 0)
+		(at 159.766 36.322 0)
 		(effects
 			(font
@@
 			)
 		)
-		(property "Footprint" "SOIC127P600X175-8N"
+		(property "Footprint" "Package_SO:SOIC-8_3.9x4.9mm_P1.27mm"
 			(at 173.99 152.07 0)
 			(effects

Commit message: Kicad fin schema
Parts:
- removed J2, J3: Conn_01x02, Connector_JST:JST_XH_B2B-XH-A_1x02_P2.50mm_Vertical, symbol Connector_Generic:Conn_01x02
Connections:
- net ADC_IN1 is gone; now on net INT: U4.6 (PA1)
- net AVDD is gone; now on net +5V: J5.7 (Pin_7)
- net PG10 is gone; now on net I2C_RST: C3.1, J6.9 (Pin_9), U4.4 (PG10)
- net +3.3V: now also IC1.3 (~{W}), IC1.7 (~{HOLD}), IC1.8 (VCC), J5.8 (Pin_8)
- net GND: now also IC1.4 (VSS)
- net LPn: now also U4.13 (PB0)
- net PWR_EN: now also U4.5 (PA0)
- net SCL: now also U4.19 (PA9)
- net SDA: now also U4.25 (PA15)
- net USART2_RX: now also U4.8 (PA3); no longer U4.5 (PA0)
- net Chip Select: now reaches IC1.1 (~{S})
- net Chip Select: now also U4.9 (PA4)
- net MISO: now reaches IC1.2 (Q)
- net MISO: now also U4.11 (PA6)
- net MOSI: now reaches IC1.5 (D)
- net MOSI: now also U4.12 (PA7)
- net SCK: now reaches IC1.6 (C)
- net SCK: now also U4.10 (PA5)
- no-connect marks 19 -> 11
Other:
- note added: "Connecteur capteur VL53L5CX-SATEL"
- note added: "EEPROM"
- note removed: "EEPROM M95512-RMN6TP"
- moved on the sheet: C3, J1, J5
